Commit message: ur5 with splited driver

File: src/arm_rviz/urdf/skai_arm.ros2_control.xacro (robot description, xacro)
@@ -6,11 +6,10 @@
             <hardware>
                 <!-- By default, set up controllers for simulation. This won't work on real hardware -->
-                <!--plugin>mock_components/GenericSystem</plugin-->
-                <plugin>skai_hardware/SKAIHardware</plugin>
+                <plugin>mock_components/GenericSystem</plugin>
             </hardware>
             <joint name="ROT_1">
                 <command_interface name="position"/>
                 <state_interface name="position">
-                  <param name="initial_value">${initial_positions['ROT_1']}</param>
+                  <param name="initial_value">0.0</param>
                 </state_interface>
             </joint>
@@ -18,5 +17,5 @@
                 <command_interface name="position"/>
                 <state_interface name="position">
-                  <param name="initial_value">${initial_positions['PITCH_1']}</param>
+                  <param name="initial_value">0.0</param>
                 </state_interface>
             </joint>
@@ -24,5 +23,5 @@
                 <command_interface name="position"/>
                 <state_interface name="position">
-                  <param name="initial_value">${initial_positions['PITCH_2']}</param>
+                  <param name="initial_value">0.0</param>
                 </state_interface>
             </joint>
@@ -30,5 +29,5 @@
                 <command_interface name="position"/>
                 <state_interface name="position">
-                  <param name="initial_value">${initial_positions['PITCH_3']}</param>
+                  <param name="initial_value">0.0</param>
                 </state_interface>
             </joint>
@@ -36,5 +35,5 @@
                 <command_interface name="position"/>
                 <state_interface name="position">
-                  <param name="initial_value">${initial_positions['ROT_2']}</param>
+                  <param name="initial_value">0.0</param>
                 </state_interface>
             </joint>
@@ -42,5 +41,5 @@
                 <command_interface name="position"/>
                 <state_interface name="position">
-                  <param name="initial_value">${initial_positions['ROT_3']}</param>
+                  <param name="initial_value">0.0</param>
                 </state_interface>
             </joint>

File: src/arm_rviz/urdf/skai_arm.urdf (robot description, URDF)
Before this commit: robot skai_arm, 7 links, 6 joints
Links:
- removed link BASE
- added link base_link, mass 49.417; collision mesh filename=package://arm_rviz/meshes/BASE.STL; visual mesh filename=package://arm_rviz/meshes/BASE.STL
- link J_5: mass 0.26391 -> 0.26474
- link J_6: mass 0.39709 -> 0.3973
Joints:
- joint PITCH_1: limit lower=-3.14 upper=0 effort=0 velocity=0 -> lower=-3.14 upper=0 effort=10 velocity=0.1; origin xyz=0 -0.0459999999999999 0.194000000000002 rpy=-1.5707963267949 0.523598775598295 0 -> xyz=0 -0.046 0.194 rpy=-1.5708 0.5236 0
- joint PITCH_2: limit lower=-2.61 upper=2.61 effort=0 velocity=0 -> lower=-2.61 upper=2.61 effort=10 velocity=0.1; origin xyz=-0.371524898223531 0.214500000000008 0.103 rpy=3.14159265358979 0 -0.523598775598295 -> xyz=-0.37152 0.2145 0.103 rpy=3.1416 0 -0.5236
- joint PITCH_3: limit lower=-6.28 upper=6.28 effort=0 velocity=0 -> lower=-3.14 upper=3.14 effort=10 velocity=0.1; origin xyz=-0.409 0 -0.016 rpy=0 0 1.9322 -> xyz=-0.408999999999995 0 -0.0160000000000003 rpy=0 0 1.93219930379001
- joint ROT_1: origin xyz=-0.067 -0.065 0.0820000000000001 rpy=0 0 0 -> xyz=0 0.012 0.082 rpy=0 0 0; parent BASE -> base_link
- joint ROT_2: axis 1 0 0 -> 0 0 -1; limit lower=-6.28 upper=6.28 effort=10 velocity=0.1 -> lower=-3.14 upper=3.14 effort=10 velocity=0.1; origin xyz=0.00088397 0.0023385 -0.0725 rpy=0 0 -1.9322 -> xyz=0.023514 0.062204 -0.0725 rpy=-1.5708 0.3614 2.7802
- joint ROT_3: axis 0 0 -1 -> 0 0 1; limit lower=-6.28 upper=6.28 effort=10 velocity=0.1 -> lower=-3.14 upper=3.14 effort=10 velocity=0.1; origin xyz=-0.139499963386566 -1.48215814215757E-05 0.347396030273288 rpy=0 0 0 -> xyz=-0.12301 -0.32542 -0.0695 rpy=1.221 -1.5708 0
